Commit message: feat: add gazebo simu

File: description/ros2_control/explorer.ros2_control.xacro (robot description, xacro)
@@ -1,8 +1,13 @@
 <?xml version="1.0"?>
 <robot xmlns:xacro="http://www.ros.org/wiki/xacro">
-  <xacro:macro name="explorer_ros2_control" params="name">
+  <xacro:macro name="explorer_ros2_control" params="name use_gazebo_classic:=^|false">
     <ros2_control name="${name}" type="system">
       <hardware>
-        <plugin>ros2_control_explorer/RobotSystem</plugin>
+        <xacro:if value="${use_gazebo_classic}">
+          <plugin>gazebo_ros2_control/GazeboSystem</plugin>
+        </xacro:if>
+        <xacro:unless value="${use_gazebo_classic}">
+          <plugin>ros2_control_explorer/RobotSystem</plugin>
+        </xacro:unless>
       </hardware>
       <joint name="joint_1">
@@ -30,5 +35,5 @@
         </command_interface>
         <state_interface name="position">
-          <param name="initial_value">0.0</param>
+          <param name="initial_value">0.5</param>
         </state_interface>
         <state_interface name="velocity"/>

File: description/urdf/explorer.urdf.xacro (robot description, xacro)
@@ -1,4 +1,5 @@
 <?xml version="1.0"?>
 <robot xmlns:xacro="http://wiki.ros.org/xacro" name="explorer">
+  <xacro:arg name="use_gazebo_classic" default="false" />
   <!-- Import explorer macro -->
   <xacro:include filename="$(find ros2_control_explorer)/description/urdf/explorer_old_description.urdf.xacro"/>
@@ -8,4 +9,9 @@
   <!-- Import explorer ros2_control description -->
   <xacro:include filename="$(find ros2_control_explorer)/description/ros2_control/explorer.ros2_control.xacro" />
-  <xacro:explorer_ros2_control name="explorer"/>
+  <xacro:explorer_ros2_control name="explorer" use_gazebo_classic="$(arg use_gazebo_classic)"/>
+  <xacro:if value="$(arg use_gazebo_classic)">
+    <!-- Import Gazebo Classic definitions + plugin -->
+    <xacro:include filename="$(find ros2_control_explorer)/description/gazebo/explorer.gazebo.xacro" />
+    <xacro:explorer_gazebo/>
+  </xacro:if>
 </robot>

File: description/urdf/explorer_new_description.urdf.xacro (robot description, xacro)
@@ -8,5 +8,5 @@
       xyz_offset="0 0 0"
       rpy_offset="0 0 0"
-      mesh_package="ros2_control_explorer/description"
+      mesh_package="ros2_control_explorer"
       mesh_name="base_link"
   />
@@ -15,5 +15,5 @@
       xyz_offset="0 0 0"
       rpy_offset="0 0 0"
-      mesh_package="ros2_control_explorer/description"
+      mesh_package="ros2_control_explorer"
       mesh_name="link1"
   />
@@ -22,5 +22,5 @@
       xyz_offset="0 0 0"
       rpy_offset="0 0 0"
-      mesh_package="ros2_control_explorer/description"
+      mesh_package="ros2_control_explorer"
       mesh_name="link2"
   />
@@ -29,5 +29,5 @@
       xyz_offset="0 0 0"
       rpy_offset="0 0 0"
-      mesh_package="ros2_control_explorer/description"
+      mesh_package="ros2_control_explorer"
       mesh_name="link3"
   />
@@ -36,5 +36,5 @@
       xyz_offset="0 0 0"
       rpy_offset="0 0 0"
-      mesh_package="ros2_control_explorer/description"
+      mesh_package="ros2_control_explorer"
       mesh_name="link4_new"
   />
@@ -43,5 +43,5 @@
       xyz_offset="0 0 0"
       rpy_offset="0 0 0"
-      mesh_package="ros2_control_explorer/description"
+      mesh_package="ros2_control_explorer"
       mesh_name="link5_new"
   />
@@ -50,5 +50,5 @@
       xyz_offset="0 0 0"
       rpy_offset="0 0 0"
-      mesh_package="ros2_control_explorer/description"
+      mesh_package="ros2_control_explorer"
       mesh_name="gripper"
   />

File: description/urdf/explorer_old_description.urdf.xacro (robot description, xacro)
@@ -8,5 +8,5 @@
       xyz_offset="0 0 0"
       rpy_offset="0 0 0"
-      mesh_package="ros2_control_explorer/description"
+      mesh_package="ros2_control_explorer"
       mesh_name="base_link"
   />
@@ -15,5 +15,5 @@
       xyz_offset="0 0 0"
       rpy_offset="0 0 0"
-      mesh_package="ros2_control_explorer/description"
+      mesh_package="ros2_control_explorer"
       mesh_name="link1"
   />
@@ -22,5 +22,5 @@
       xyz_offset="0 0 0"
       rpy_offset="0 0 0"
-      mesh_package="ros2_control_explorer/description"
+      mesh_package="ros2_control_explorer"
       mesh_name="link2"
   />
@@ -29,5 +29,5 @@
       xyz_offset="0 0 0"
       rpy_offset="0 0 0"
-      mesh_package="ros2_control_explorer/description"
+      mesh_package="ros2_control_explorer"
       mesh_name="link3"
   />
@@ -36,5 +36,5 @@
       xyz_offset="0 0 0"
       rpy_offset="0 0 0"
-      mesh_package="ros2_control_explorer/description"
+      mesh_package="ros2_control_explorer"
       mesh_name="link4_old"
   />
@@ -43,5 +43,5 @@
       xyz_offset="0 0 0"
       rpy_offset="0 0 0"
-      mesh_package="ros2_control_explorer/description"
+      mesh_package="ros2_control_explorer"
       mesh_name="link5_old"
   />
@@ -50,5 +50,5 @@
       xyz_offset="0 0 0"
       rpy_offset="0 0 0"
-      mesh_package="ros2_control_explorer/description"
+      mesh_package="ros2_control_explorer"
       mesh_name="gripper"
   />

File: description/urdf/inc/create_link.xacro (robot description, xacro)
@@ -11,5 +11,5 @@
         <origin xyz="${xyz_offset}" rpy="${rpy_offset}"/>
         <geometry>
-          <mesh filename="package://${mesh_package}/meshes/visual/${mesh_name}.dae"/>
+          <mesh filename="file://$(find ${mesh_package})/description/meshes/visual/${mesh_name}.dae"/>
         </geometry>
       </visual>
@@ -17,5 +17,5 @@
         <origin xyz="${xyz_offset}" rpy="${rpy_offset}"/>
         <geometry>
-          <mesh filename="package://${mesh_package}/meshes/collision/${mesh_name}.stl"/>
+          <mesh filename="file://$(find ${mesh_package})/description/meshes/collision/${mesh_name}.stl"/>
         </geometry>
       </collision>

File: explorer.urdf (robot description, URDF)
Before this commit: robot explorer, 10 links, 9 joints
Links:
- link base_link: geometry collision mesh filename=file:///home/orthopus/explorer_ws/install/ros2_control_expl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; visual mesh filename=file:///home/orthopus/explorer_ws/install/ros2_control_expl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
- link link_1: geometry collision mesh filename=file:///home/orthopus/explorer_ws/install/ros2_control_expl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; visual mesh filename=file:///home/orthopus/explorer_ws/install/ros2_control_expl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
- link link_2: geometry collision mesh filename=file:///home/orthopus/explorer_ws/install/ros2_control_expl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; visual mesh filename=file:///home/orthopus/explorer_ws/install/ros2_control_expl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
- link link_3: geometry collision mesh filename=file:///home/orthopus/explorer_ws/install/ros2_control_expl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; visual mesh filename=file:///home/orthopus/explorer_ws/install/ros2_control_expl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
- link link_4: geometry collision mesh filename=file:///home/orthopus/explorer_ws/install/ros2_control_expl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; visual mesh filename=file:///home/orthopus/explorer_ws/install/ros2_control_expl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
- link link_5: geometry collision mesh filename=file:///home/orthopus/explorer_ws/install/ros2_control_expl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; visual mesh filename=file:///home/orthopus/explorer_ws/install/ros2_control_expl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
- link link_6: geometry collision mesh filename=file:///home/orthopus/explorer_ws/install/ros2_control_expl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; visual mesh filename=file:///home/orthopus/explorer_ws/install/ros2_control_expl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

Commit message: fix: circular trajectory

File: description/ros2_control/explorer.ros2_control.xacro (robot description, xacro)
@@ -35,5 +35,5 @@
         </command_interface>
         <state_interface name="position">
-          <param name="initial_value">0.5</param>
+          <param name="initial_value">0.0</param>
         </state_interface>
         <state_interface name="velocity"/>
@@ -95,12 +95,4 @@
         <state_interface name="velocity"/>
       </joint>
-      <sensor name="tcp_fts_sensor">
-        <state_interface name="force.x"/>
-        <state_interface name="force.y"/>
-        <state_interface name="force.z"/>
-        <state_interface name="torque.x"/>
-        <state_interface name="torque.y"/>
-        <state_interface name="torque.z"/>
-      </sensor>
     </ros2_control>
   </xacro:macro>

File: description/urdf/explorer_new_description.urdf.xacro (robot description, xacro)
@@ -1,5 +1,5 @@
 <?xml version="1.0"?>
 <robot xmlns:xacro="http://www.ros.org/wiki/xacro">
-  <xacro:macro name="explorer_old_description">
+  <xacro:macro name="explorer_new_description">
   <!-- helper macro -->
   <xacro:include filename="$(find ros2_control_explorer)/description/urdf/inc/create_link.xacro"/>
@@ -73,5 +73,5 @@
     <parent link="link_1"/>
     <child link="link_2"/>
-    <origin xyz="0 24.5 58.952" rpy="${pi/2} 0 0"/>
+    <origin xyz="0 24.5 58.952" rpy="${pi/2} ${-pi/2} 0"/>
     <axis xyz="0 0 1"/>
     <limit effort="1000.0" lower="0" upper="${pi}" velocity="2.5"/>
@@ -80,5 +80,5 @@
     <parent link="link_2"/>
     <child link="link_3"/>
-    <origin xyz="409.872 0 -2" rpy="${pi} 0 0"/>
+    <origin xyz="409.872 0 -2" rpy="${pi} 0 ${-pi/2}"/>
     <axis xyz="0 0 1"/>
     <limit effort="1000.0" lower="${-pi}" upper="${pi}" velocity="2.5"/>

File: description/urdf/explorer_old_description.urdf.xacro (robot description, xacro)
@@ -73,12 +73,12 @@
     <parent link="link_1"/>
     <child link="link_2"/>
-    <origin xyz="0 24.5 58.952" rpy="${pi/2} 0 0"/>
+    <origin xyz="0 24.5 58.952" rpy="${pi/2} ${-pi/2} 0"/>
     <axis xyz="0 0 1"/>
-    <limit effort="1000.0" lower="0" upper="${pi}" velocity="2.5"/>
+    <limit effort="1000.0" lower="${-pi/2}" upper="${pi/2}" velocity="2.5"/>
   </joint>
   <joint name="joint_3" type="revolute">
     <parent link="link_2"/>
     <child link="link_3"/>
-    <origin xyz="409.872 0 -2" rpy="${pi} 0 0"/>
+    <origin xyz="409.872 0 -2" rpy="${pi} 0 ${-pi/2}"/>
     <axis xyz="0 0 1"/>
     <limit effort="1000.0" lower="${-pi}" upper="${pi}" velocity="2.5"/>
