Commit message: (feat): start adding cartesian control

File: ros2_control_explorer/description/urdf/explorer_new_description.urdf.xacro (robot description, xacro)
@@ -75,5 +75,5 @@
     <origin xyz="0 24.5 58.952" rpy="${pi/2} ${-pi/2} 0"/>
     <axis xyz="0 0 1"/>
-    <limit effort="1000.0" lower="0" upper="${pi}" velocity="2.5"/>
+    <limit effort="1000.0" lower="${-pi/2}" upper="${pi/2}" velocity="2.5"/>
   </joint>
   <joint name="joint_3" type="revolute">

Commit message: (fix): scale URDF

File: ros2_control_explorer/description/urdf/explorer_new_description.urdf.xacro (robot description, xacro)
@@ -66,5 +66,5 @@
     <parent link="base_link"/>
     <child link="link_1"/>
-    <origin xyz="0 0 55.5" rpy="0 0 0"/>
+    <origin xyz="0 0 0.0555" rpy="0 0 0"/>
     <axis xyz="0 0 1"/>
     <limit effort="1000.0" lower="${-pi}" upper="${pi}" velocity="2.5"/>
@@ -73,5 +73,5 @@
     <parent link="link_1"/>
     <child link="link_2"/>
-    <origin xyz="0 24.5 58.952" rpy="${pi/2} ${-pi/2} 0"/>
+    <origin xyz="0 0.0245 0.058952" rpy="${pi/2} ${-pi/2} 0"/>
     <axis xyz="0 0 1"/>
     <limit effort="1000.0" lower="${-pi/2}" upper="${pi/2}" velocity="2.5"/>
@@ -80,12 +80,12 @@
     <parent link="link_2"/>
     <child link="link_3"/>
-    <origin xyz="409.872 0 -2" rpy="${pi} 0 ${-pi/2}"/>
+    <origin xyz="0.409872 0 -0.002" rpy="${pi} 0 ${-pi/2}"/>
     <axis xyz="0 0 1"/>
-    <limit effort="1000.0" lower="${-pi}" upper="${pi}" velocity="2.5"/>
+    <limit effort="1000.0" lower="${-3*pi/2}" upper="${pi/2}" velocity="2.5"/>
   </joint>
   <joint name="joint_4" type="revolute">
     <parent link="link_3"/>
     <child link="link_4"/>
-    <origin xyz="233.9 0 -14" rpy="0 ${pi/2} 0"/>
+    <origin xyz="0.2339 0 -0.014" rpy="0 ${pi/2} 0"/>
     <axis xyz="0 0 1"/>
     <limit effort="1000.0" lower="${-pi}" upper="${pi}" velocity="2.5"/>
@@ -94,5 +94,5 @@
     <parent link="link_4"/>
     <child link="link_5"/>
-    <origin xyz="29.593 0 92.149" rpy="$0 ${pi/2} 0"/>
+    <origin xyz="0.029593 0 0.092149" rpy="0 ${pi/2} 0"/>
     <axis xyz="0 0 1"/>
     <limit effort="1000.0" lower="${-pi}" upper="${pi}" velocity="2.5"/>
@@ -101,5 +101,5 @@
     <parent link="link_5"/>
     <child link="link_6"/>
-    <origin xyz="-150.049 0 -28.307" rpy="0 ${-pi/2} 0"/>
+    <origin xyz="-0.150049 0 -0.028307" rpy="0 ${-pi/2} 0"/>
     <axis xyz="0 0 1"/>
     <limit effort="1000.0" lower="${-pi}" upper="${pi}" velocity="2.5"/>

File: ros2_control_explorer/description/urdf/explorer_old_description.urdf.xacro (robot description, xacro)
@@ -66,5 +66,5 @@
     <parent link="base_link"/>
     <child link="link_1"/>
-    <origin xyz="0 0 55.5" rpy="0 0 0"/>
+    <origin xyz="0 0 0.0555" rpy="0 0 0"/>
     <axis xyz="0 0 1"/>
     <limit effort="1000.0" lower="${-pi}" upper="${pi}" velocity="2.5"/>
@@ -73,5 +73,5 @@
     <parent link="link_1"/>
     <child link="link_2"/>
-    <origin xyz="0 24.5 58.952" rpy="${pi/2} ${-pi/2} 0"/>
+    <origin xyz="0 0.0245 0.058952" rpy="${pi/2} ${-pi/2} 0"/>
     <axis xyz="0 0 1"/>
     <limit effort="1000.0" lower="${-pi/2}" upper="${pi/2}" velocity="2.5"/>
@@ -80,12 +80,12 @@
     <parent link="link_2"/>
     <child link="link_3"/>
-    <origin xyz="409.872 0 -2" rpy="${pi} 0 ${-pi/2}"/>
+    <origin xyz="0.409872 0 -0.002" rpy="${pi} 0 ${-pi/2}"/>
     <axis xyz="0 0 1"/>
-    <limit effort="1000.0" lower="${-pi}" upper="${pi}" velocity="2.5"/>
+    <limit effort="1000.0" lower="${-3*pi/2}" upper="${pi/2}" velocity="2.5"/>
   </joint>
   <joint name="joint_4" type="revolute">
     <parent link="link_3"/>
     <child link="link_4"/>
-    <origin xyz="233.9 0 -14" rpy="0 ${pi/2} 0"/>
+    <origin xyz="0.2339 0 -0.014" rpy="0 ${pi/2} 0"/>
     <axis xyz="0 0 1"/>
     <limit effort="1000.0" lower="${-pi}" upper="${pi}" velocity="2.5"/>
@@ -94,5 +94,5 @@
     <parent link="link_4"/>
     <child link="link_5"/>
-    <origin xyz="0 90 83" rpy="${(65*pi)/180} 0 ${pi}"/>
+    <origin xyz="0 0.090 0.083" rpy="${(65*pi)/180} 0 ${pi}"/>
     <axis xyz="0 0 1"/>
     <limit effort="1000.0" lower="${-pi}" upper="${pi}" velocity="2.5"/>
@@ -101,5 +101,5 @@
     <parent link="link_5"/>
     <child link="link_6"/>
-    <origin xyz="0 90 83" rpy="${-(65*pi)/180} 0 0"/>
+    <origin xyz="0 0.090 0.083" rpy="${-(65*pi)/180} 0 0"/>
     <axis xyz="0 0 1"/>
     <limit effort="1000.0" lower="${-pi}" upper="${pi}" velocity="2.5"/>

File: ros2_control_explorer/description/urdf/inc/create_link.xacro (robot description, xacro)
@@ -11,5 +11,5 @@
         <origin xyz="${xyz_offset}" rpy="${rpy_offset}"/>
         <geometry>
-          <mesh filename="file://$(find ${mesh_package})/description/meshes/visual/${mesh_name}.dae"/>
+          <mesh filename="file://$(find ${mesh_package})/description/meshes/visual/${mesh_name}.dae" scale="0.001 0.001 0.001"/>
         </geometry>
       </visual>
@@ -17,5 +17,5 @@
         <origin xyz="${xyz_offset}" rpy="${rpy_offset}"/>
         <geometry>
-          <mesh filename="file://$(find ${mesh_package})/description/meshes/collision/${mesh_name}.stl"/>
+          <mesh filename="file://$(find ${mesh_package})/description/meshes/collision/${mesh_name}.stl" scale="0.001 0.001 0.001"/>
         </geometry>
       </collision>

Commit message: (feat): Add mass and inertia (WIP)

File: ros2_control_explorer/description/urdf/explorer_new_description.urdf.xacro (robot description, xacro)
@@ -10,4 +10,12 @@
       mesh_package="ros2_control_explorer"
       mesh_name="base_link"
+      xyz_mass="0 0 0"
+      mass="1"
+      ixx="1"
+      ixy="0"
+      ixz="0"
+      iyy="1"
+      iyz="0"
+      izz="1"
   />
   <xacro:create_link
@@ -17,4 +25,12 @@
       mesh_package="ros2_control_explorer"
       mesh_name="link1"
+      xyz_mass="0 0 0"
+      mass="1"
+      ixx="1"
+      ixy="0"
+      ixz="0"
+      iyy="1"
+      iyz="0"
+      izz="1"
   />
   <xacro:create_link
@@ -24,4 +40,12 @@
       mesh_package="ros2_control_explorer"
       mesh_name="link2"
+      xyz_mass="0 0 0"
+      mass="1"
+      ixx="1"
+      ixy="0"
+      ixz="0"
+      iyy="1"
+      iyz="0"
+      izz="1"
   />
   <xacro:create_link
@@ -31,4 +55,12 @@
       mesh_package="ros2_control_explorer"
       mesh_name="link3"
+      xyz_mass="0 0 0"
+      mass="1"
+      ixx="1"
+      ixy="0"
+      ixz="0"
+      iyy="1"
+      iyz="0"
+      izz="1"
   />
   <xacro:create_link
@@ -38,4 +70,12 @@
       mesh_package="ros2_control_explorer"
       mesh_name="link4_new"
+      xyz_mass="0 0 0"
+      mass="1"
+      ixx="1"
+      ixy="0"
+      ixz="0"
+      iyy="1"
+      iyz="0"
+      izz="1"
   />
   <xacro:create_link
@@ -45,4 +85,12 @@
       mesh_package="ros2_control_explorer"
       mesh_name="link5_new"
+      xyz_mass="0 0 0"
+      mass="1"
+      ixx="1"
+      ixy="0"
+      ixz="0"
+      iyy="1"
+      iyz="0"
+      izz="1"
   />
   <xacro:create_link
@@ -52,4 +100,12 @@
       mesh_package="ros2_control_explorer"
       mesh_name="gripper"
+      xyz_mass="0 0 0"
+      mass="1"
+      ixx="1"
+      ixy="0"
+      ixz="0"
+      iyy="1"
+      iyz="0"
+      izz="1"
   />
   <link name="ft_frame"/>

File: ros2_control_explorer/description/urdf/explorer_old_description.urdf.xacro (robot description, xacro)
@@ -10,4 +10,12 @@
       mesh_package="ros2_control_explorer"
       mesh_name="base_link"
+      xyz_mass="0.000045 0.000001 0.026873"
+      mass="0.520"
+      ixx="369892.299"
+      ixy="-216.179"
+      ixz="263.279"
+      iyy="366673.241"
+      iyz="13.226"
+      izz="433449.993"
   />
   <xacro:create_link
@@ -17,4 +25,12 @@
       mesh_package="ros2_control_explorer"
       mesh_name="link1"
+      xyz_mass="-0.000001 0.02935 0.029854"
+      mass="0.318"
+      ixx="323959.935"
+      ixy="3.991"
+      ixz="9.773"
+      iyy="322143.455"
+      iyz="-86000.965"
+      izz="237019.412"
   />
   <xacro:create_link
@@ -24,4 +40,12 @@
       mesh_package="ros2_control_explorer"
       mesh_name="link2"
+      xyz_mass="0.204774 0.000012 0.057505"
+      mass="2.023"
+      ixx="2433042.798"
+      ixy="194.199"
+      ixz="1567.055"
+      iyy="57628887.234"
+      iyz="566.556"
+      izz="28172.073"
   />
   <xacro:create_link
@@ -31,4 +55,12 @@
       mesh_package="ros2_control_explorer"
       mesh_name="link3"
+      xyz_mass="0.138064 -0.000019  -0.007584"
+      mass="1.074"
+      ixx="563205.607"
+      ixy="1291.964"
+      ixz="588051.397"
+      iyy="6043403.387"
+      iyz="169.302"
+      izz="6205261.854"
   />
   <xacro:create_link
@@ -38,4 +70,12 @@
       mesh_package="ros2_control_explorer"
       mesh_name="link4_old"
+      xyz_mass="0.000006 0.044695  0.057883"
+      mass="0.687"
+      ixx="1204142.247"
+      ixy="-1088.536"
+      ixz="-428.569"
+      iyy="794422.875"
+      iyz="-320135.516"
+      izz="929643.790"
   />
   <xacro:create_link
@@ -45,4 +85,12 @@
       mesh_package="ros2_control_explorer"
       mesh_name="link5_old"
+      xyz_mass="0.000006 0.044695  0.057883"
+      mass="0.687"
+      ixx="1204142.247"
+      ixy="-1088.536"
+      ixz="-428.569"
+      iyy="794422.875"
+      iyz="-320135.516"
+      izz="929643.790"
   />
   <xacro:create_link
@@ -52,4 +100,12 @@
       mesh_package="ros2_control_explorer"
       mesh_name="gripper"
+      xyz_mass="0.00224 -0.000032 0.077277"
+      mass="0.407"
+      ixx="1506746.748"
+      ixy="931.438"
+      ixz="-95753.657"
+      iyy="1072546.483"
+      iyz="273.718"
+      izz="713799.995"
   />
   <link name="ft_frame"/>
@@ -108,5 +164,5 @@
     <parent link="link_6"/>
     <child link="ft_frame"/>
-    <origin xyz="0 0 0" rpy="0 0 0"/>
+    <origin xyz="0.011 0 0.15" rpy="0 0 0"/>
   </joint>
   <joint name="joint-tool" type="fixed">

File: ros2_control_explorer/description/urdf/inc/create_link.xacro (robot description, xacro)
@@ -6,5 +6,13 @@
         rpy_offset
         mesh_package
-        mesh_name">
+        mesh_name
+        xyz_mass
+        mass
+        ixx
+        ixy
+        ixz
+        iyy
+        iyz
+        izz">
     <link name="${link_name}">
       <visual>
@@ -21,6 +29,7 @@
       </collision>
       <inertial>
-        <mass value="1"/>
-        <inertia ixx="1.0" ixy="0.0" ixz="0.0" iyy="1.0" iyz="0.0" izz="1.0"/>
+        <origin xyz="${xyz_mass}" rpy="0 0 0"/>
+        <mass value="${mass}"/>
+        <inertia ixx="${ixx}" ixy="${ixy}" ixz="${ixz}" iyy="${iyy}" iyz="${iyz}" izz="${izz}"/>
       </inertial>
     </link>
