Commit message: (fix) : modification urdf wheelchair

File: ros2_control_wheelchair/description/urdf/wheelchair.urdf.xacro (robot description, xacro)
@@ -4,5 +4,5 @@
  <!-- Import Rviz colors -->
   <xacro:include filename="$(find ros2_control_wheelchair)/description/material/wheelchair.materials.xacro" />
-  <xacro:include filename="$(find ros2_control_wheelchair)/description/urdf/wheelchair_description_test.urdf.xacro" />
+  <xacro:include filename="$(find ros2_control_wheelchair)/description/urdf/wheelchair_description.urdf.xacro" />
   <!-- Import wheelchair ros2_control description -->
   <xacro:include filename="$(find ros2_control_wheelchair)/description/ros2_control/wheelchair.ros2_control.xacro" />

File: ros2_control_wheelchair/description/urdf/wheelchair_description.urdf.xacro (robot description, xacro)
@@ -4,26 +4,26 @@
   <link name="chassis">
       <collision>
-        <origin xyz="-0.151427 -0 0.5" rpy="0 0 0"/>
-        <geometry>
-          <box size="2.01142 1 0.568726"/>
-        </geometry>
-      </collision>
-      <visual>
-        <origin xyz="-0.151427 -0 0.5" rpy="0 0 0"/>
-        <geometry>
-          <box size="2.01142 1 0.568726"/>
+        <origin xyz="0 0 0.225" rpy="0 0 0"/>
+        <geometry>
+          <box size="0.6 0.5 0.25"/>
+        </geometry>
+      </collision>
+      <visual>
+        <origin xyz="0 0 0.225" rpy="0 0 0"/>
+        <geometry>
+          <box size="0.6 0.5 0.25"/>
         </geometry>
         <material name="orange"/>
       </visual>
       <inertial>
-        <origin xyz="-0.151427 -0 0.5" rpy="0 0 0"/>
-        <mass value="1.14395"/>
-        <inertia
-          ixx="0.126164"
-          ixy="0.0"
-          ixz="0.0"
-          iyy="0.416519"
-          iyz="0.0"
-          izz="0.481014"/>
+        <origin xyz="0.0 0.0 0.225" rpy="0 0 0"/>
+        <mass value="70"/>
+        <inertia
+          ixx="1.82291666667"
+          ixy="0.0"
+          ixz="0.0"
+          iyy="2.46458333333"
+          iyz="0.0"
+          izz="3.55833333333"/>
       </inertial>
     </link>
@@ -32,28 +32,114 @@
       <collision>
         <geometry>
-          <cylinder length="0.08" radius="0.3" />
-        </geometry>
-      </collision>
-      <visual>
-        <geometry>
-          <cylinder length="0.08" radius="0.3" />
+          <cylinder length="0.09" radius="0.175" />
+        </geometry>
+      </collision>
+      <visual>
+        <geometry>
+          <cylinder length="0.09" radius="0.175" />
         </geometry>
         <material name="black" />
       </visual>
       <inertial>
+        <mass value="5" />
+        <inertia ixx="0.041656" ixy="0.0" ixz="0.0" iyy="0.041656" iyz="0.0" izz="0.0765625" />
+      </inertial>
+    </link>
+     <!-- right wheel Link -->
+    <link name="right_wheel">
+      <collision>
+        <geometry>
+          <cylinder length="0.09" radius="0.175" />
+        </geometry>
+      </collision>
+      <visual>
+        <geometry>
+          <cylinder length="0.09" radius="0.175" />
+        </geometry>
+        <material name="black" />
+      </visual>
+      <inertial>
+        <mass value="5" />
+        <inertia ixx="0.041656" ixy="0.0" ixz="0.0" iyy="0.041656" iyz="0.0" izz="0.0765625" />
+      </inertial>
+    </link>
+    <link name="fixation_front_left">
+      <collision>
+        <origin xyz="0 0 0" rpy="0 0 0"/>
+        <geometry>
+          <box size="0.2 0.025 0.04"/>
+        </geometry>
+      </collision>
+      <visual>
+        <origin xyz="0 0 0" rpy="0 0 0"/>
+        <geometry>
+          <box size="0.2 0.025 0.04"/>
+        </geometry>
+        <material name="orange"/>
+      </visual>
+      <inertial>
+        <origin xyz="0 0 0" rpy="0 0 0"/>
+        <mass value="0.5"/>
+        <inertia
+          ixx="0.00009270833"
+          ixy="0.0"
+          ixz="0.0"
+          iyy="0.00173333333"
+          iyz="0.0"
+          izz="0.00169270833"/>
+      </inertial>
+    </link>
+    <link name="left_front_wheel">
+      <collision>
+        <geometry>
+          <cylinder length="0.09" radius="0.085" />
+        </geometry>
+      </collision>
+      <visual>
+        <geometry>
+          <cylinder length="0.09" radius="0.085" />
+        </geometry>
+        <material name="black" />
+      </visual>
+      <inertial>
         <mass value="2" />
-        <inertia ixx="0.145833" ixy="0.0" ixz="0.0" iyy="0.145833" iyz="0.0" izz="0.125" />
-      </inertial>
-    </link>
-    <!-- right wheel Link -->
-    <link name="right_wheel">
-      <collision>
-        <geometry>
-          <cylinder length="0.08" radius="0.3" />
-        </geometry>
-      </collision>
-      <visual>
-        <geometry>
-          <cylinder length="0.08" radius="0.3" />
+        <inertia ixx="0.0049625" ixy="0.0" ixz="0.0" iyy="0.0049625" iyz="0.0" izz="0.007225" />
+      </inertial>
+    </link>
+    <link name="fixation_front_right">
+      <collision>
+        <origin xyz="0 0 0" rpy="0 0 0"/>
+        <geometry>
+          <box size="0.2 0.025 0.04"/>
+        </geometry>
+      </collision>
+      <visual>
+        <origin xyz="0 0 0" rpy="0 0 0"/>
+        <geometry>
+          <box size="0.2 0.025 0.04"/>
+        </geometry>
+        <material name="orange"/>
+      </visual>
+      <inertial>
+        <origin xyz="0 0 0" rpy="0 0 0"/>
+        <mass value="0.5"/>
+        <inertia
+          ixx="0.00009270833"
+          ixy="0.0"
+          ixz="0.0"
+          iyy="0.00173333333"
+          iyz="0.0"
+          izz="0.00169270833"/>
+      </inertial>
+    </link>
+    <link name="right_front_wheel">
+      <collision>
+        <geometry>
+          <cylinder length="0.09" radius="0.085" />
+        </geometry>
+      </collision>
+      <visual>
+        <geometry>
+          <cylinder length="0.09" radius="0.085" />
         </geometry>
         <material name="black" />
@@ -61,50 +147,416 @@
       <inertial>
         <mass value="2" />
-        <inertia ixx="0.145833" ixy="0.0" ixz="0.0" iyy="0.145833" iyz="0.0" izz="0.125" />
-      </inertial>
-    </link>
-    <!-- caster frontal wheel Link -->
-    <link name="caster">
-      <collision>
-        <geometry>
-          <sphere radius="0.2"/>
-        </geometry>
-      </collision>
-      <visual>
-        <geometry>
-          <sphere radius="0.2"/>
-        </geometry>
-        <material name="white"/>
-      </visual>
-      <inertial>
-        <origin xyz="-0.957138 -0 0.2" rpy="0 0 0"/>
-        <mass value="0.005"/>
-        <inertia
-          ixx="0.1"
-          ixy="0.0"
-          ixz="0.0"
-          iyy="0.1"
-          iyz="0.0"
-          izz="0.1"/>
+        <inertia ixx="0.0049625" ixy="0.0" ixz="0.0" iyy="0.0049625" iyz="0.0" izz="0.007225" />
+      </inertial>
+    </link>
+    <link name="fixation_rear_left">
+      <collision>
+        <origin xyz="0 0 0" rpy="0 0 0"/>
+        <geometry>
+          <box size="0.25 0.025 0.04"/>
+        </geometry>
+      </collision>
+      <visual>
+        <origin xyz="0 0 0" rpy="0 0 0"/>
+        <geometry>
+          <box size="0.25 0.025 0.04"/>
+        </geometry>
+        <material name="orange"/>
+      </visual>
+      <inertial>
+        <origin xyz="0 0 0" rpy="0 0 0"/>
+        <mass value="0.55"/>
+        <inertia
+          ixx="0.00010197916"
+          ixy="0.0"
+          ixz="0.0"
+          iyy="0.00293791666"
+          iyz="0.0"
+          izz="0.00289322916"/>
+      </inertial>
+    </link>
+    <link name="left_rear_wheel">
+      <collision>
+        <geometry>
+          <cylinder length="0.09" radius="0.085" />
+        </geometry>
+      </collision>
+      <visual>
+        <geometry>
+          <cylinder length="0.09" radius="0.085" />
+        </geometry>
+        <material name="black" />
+      </visual>
+      <inertial>
+        <mass value="2" />
+        <inertia ixx="0.0049625" ixy="0.0" ixz="0.0" iyy="0.0049625" iyz="0.0" izz="0.007225" />
+      </inertial>
+    </link>
+    <link name="fixation_rear_right">
+      <collision>
+        <origin xyz="0 0 0" rpy="0 0 0"/>
+        <geometry>
+          <box size="0.25 0.025 0.04"/>
+        </geometry>
+      </collision>
+      <visual>
+        <origin xyz="0 0 0" rpy="0 0 0"/>
+        <geometry>
+          <box size="0.25 0.025 0.04"/>
+        </geometry>
+        <material name="orange"/>
+      </visual>
+      <inertial>
+        <origin xyz="0 0 0" rpy="0 0 0"/>
+        <mass value="0.55"/>
+        <inertia
+          ixx="0.00010197916"
+          ixy="0.0"
+          ixz="0.0"
+          iyy="0.00293791666"
+          iyz="0.0"
+          izz="0.00289322916"/>
+      </inertial>
+    </link>
+    <link name="right_rear_wheel">
+      <collision>
+        <geometry>
+          <cylinder length="0.09" radius="0.085" />
+        </geometry>
+      </collision>
+      <visual>
+        <geometry>
+          <cylinder length="0.09" radius="0.085" />
+        </geometry>
+        <material name="black" />
+      </visual>
+      <inertial>
+        <mass value="2" />
+        <inertia ixx="0.0049625" ixy="0.0" ixz="0.0" iyy="0.0049625" iyz="0.0" izz="0.007225" />
+      </inertial>
+    </link>
+    <link name="seat_fixation">
+      <collision>
+        <origin xyz="0 0 0" rpy="0 0 0"/>
+        <geometry>
+          <box size="0.48 0.22 0.10"/>
+        </geometry>
+      </collision>
+      <visual>
+        <origin xyz="0 0 0" rpy="0 0 0"/>
+        <geometry>
+          <box size="0.48 0.22 0.10"/>
+        </geometry>
+        <material name="black"/>
+      </visual>
+      <inertial>
+        <origin xyz="0.0 0.0 0.0" rpy="0 0 0"/>
+        <mass value="3"/>
+        <inertia
+          ixx="0.0146"
+          ixy="0.0"
+          ixz="0.0"
+          iyy="0.0601"
+          iyz="0.0"
+          izz="0.0697"/>
+      </inertial>
+    </link>
+    <link name="seat">
+      <collision>
+        <origin xyz="0 0 0" rpy="0 0 0"/>
+        <geometry>
+          <box size="0.58 0.58 0.04"/>
+        </geometry>
+      </collision>
+      <visual>
+        <origin xyz="0 0 0" rpy="0 0 0"/>
+        <geometry>
+          <box size="0.58 0.58 0.04"/>
+        </geometry>
+        <material name="black"/>
+      </visual>
+      <inertial>
+        <origin xyz="0.0 0.0 0.0" rpy="0 0 0"/>
+        <mass value="3"/>
+        <inertia
+          ixx="0.0845"
+          ixy="0.0"
+          ixz="0.0"
+          iyy="0.0845"
+          iyz="0.0"
+          izz="0.1682"/>
+      </inertial>
+    </link>
+    <link name="foam_seat">
+      <visual>
+        <origin rpy="0 0 0" xyz="0 0 0"/>
+        <geometry>
+          <mesh filename="file:///home/orthopus/explorer_ws/install/ros2_control_wheelchair/share/ros2_control_wheelchair/description/meshes/visual/seat.dae" scale="0.001 0.001 0.001"/>
+        </geometry>
+      </visual>
+      <collision>
+        <origin rpy="0 0 0" xyz="0 0 0"/>
+        <geometry>
+          <mesh filename="file:///home/orthopus/explorer_ws/install/ros2_control_wheelchair/share/ros2_control_wheelchair/description/meshes/collision/seat.stl" scale="0.001 0.001 0.001"/>
+        </geometry>
+      </collision>
+      <inertial>
+        <origin rpy="0 0 0" xyz="0 -0.15 0"/>
+        <mass value="1"/>
+        <inertia ixx="0.02440833332" ixy="0" ixz="0" iyy="0.02270833332" iyz="0" izz="0.04336666666"/>
+      </inertial>
+    </link>
+    <link name="backrest_fixation">
+      <collision>
+        <origin xyz="0 0 0" rpy="0 0 0"/>
+        <geometry>
+          <box size="0.05 0.1 0.75"/>
+        </geometry>
+      </collision>
+      <visual>
+        <origin xyz="0 0 0" rpy="0 0 0"/>
+        <geometry>
+          <box size="0.05 0.1 0.75"/>
+        </geometry>
+        <material name="black"/>
+      </visual>
+      <inertial>
+        <origin xyz="0.0 0.0 0.0" rpy="0 0 0"/>
+        <mass value="3"/>
+        <inertia
+          ixx="0.143125"
+          ixy="0.0"
+          ixz="0.0"
+          iyy="0.14125"
+          iyz="0.0"
+          izz="0.003125"/>
+      </inertial>
+    </link>
+    <link name="foam_backrest">
+      <visual>
+        <origin rpy="0 0 0" xyz="0 0 0"/>
+        <geometry>
+          <mesh filename="file:///home/orthopus/explorer_ws/install/ros2_control_wheelchair/share/ros2_control_wheelchair/description/meshes/visual/backrest.dae" scale="0.001 0.001 0.001"/>
+        </geometry>
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