Commit message: (feat): add disabled simulator

File: ros2_control_explorer/description/gazebo/explorer.gazebo.xacro (robot description, xacro)
@@ -8,5 +8,5 @@
     <!-- ros_control plugin -->
     <gazebo>
-      <plugin filename="libgazebo_ros2_control.so" name="gazebo_ros2_control">
+      <plugin filename="libgazebo_ros2_control.so" name="gazebo_ros2_control_explorer">
         <parameters>$(find ros2_control_explorer)/config/explorer_controller.yaml</parameters>
       </plugin>

File: ros2_control_explorer/description/urdf/explorer.urdf.xacro (robot description, xacro)
@@ -5,5 +5,5 @@
   <xacro:include filename="$(find ros2_control_explorer)/description/urdf/explorer_old_description.urdf.xacro"/>
   <!-- create link fixed to the "world" -->
-  <link name="world"/>
+  <!-- <link name="world"/> -->
   <xacro:explorer_old_description/>
   <!-- Import explorer ros2_control description -->

File: ros2_control_explorer/description/urdf/explorer_old_description.urdf.xacro (robot description, xacro)
@@ -112,10 +112,10 @@
   <link name="tool0"/>
   <!-- base_joint fixes base_link to the environment -->
-  <joint name="base_joint" type="fixed">
+  <!-- <joint name="base_joint" type="fixed">
     <parent link="world"/>
     <child link="base_link"/>
     <origin xyz="0 0 0" rpy="0 0 0"/>
     <axis xyz="0 0 1"/>
-  </joint>
+  </joint> -->
   <!-- joints - main serial chain -->
   <joint name="joint_1" type="revolute">

File: ros2_control_wheelchair/description/gazebo/wheelchair.gazebo.xacro (robot description, xacro)
@@ -9,5 +9,5 @@
   <gazebo>
     <!-- Joint state publisher -->
-    <plugin filename="libgazebo_ros2_control.so" name="gazebo_ros2_control">
+    <plugin filename="libgazebo_ros2_control.so" name="gazebo_ros2_control_wheelchair">
       <parameters>$(find ros2_control_wheelchair)/config/wheelchair_controllers.yaml</parameters>
     </plugin>

File: ros2_control_wheelchair/description/urdf/wheelchair.urdf.xacro (robot description, xacro)
@@ -1,4 +1,3 @@
 <?xml version="1.0"?>
-<!-- 4 Wheel Robot with front steering and rear drive -->
 <robot xmlns:xacro="http://www.ros.org/wiki/xacro" name="wheelchair">
  <!-- Import Rviz colors -->
