Commit message: (fix): change meshes path

File: disabled_simulator/description/urdf/simulation.urdf.xacro (robot description, xacro)
@@ -7,5 +7,5 @@
       <origin rpy="0 0 0" xyz="0 0 0"/>
       <geometry>
-        <mesh filename="file:///home/orthopus/explorer_ws/install/disabled_simulator/share/disabled_simulator/description/meshes/visual/fixation.dae" scale="0.001 0.001 0.001"/>
+        <mesh filename="file://$(find disabled_simulator)/description/meshes/visual/fixation.dae" scale="0.001 0.001 0.001"/>
       </geometry>
     </visual>
@@ -13,5 +13,5 @@
       <origin rpy="0 0 0" xyz="0 0 0"/>
       <geometry>
-        <mesh filename="file:///home/orthopus/explorer_ws/install/disabled_simulator/share/disabled_simulator/description/meshes/collision/fixation.stl" scale="0.001 0.001 0.001"/>
+        <mesh filename="file://$(find disabled_simulator)/description/meshes/collision/fixation.stl" scale="0.001 0.001 0.001"/>
       </geometry>
     </collision>
