Commit message: (feat): add gripper pincette

File: explorer_on_wheelchair/description/ros2_control/simulation.ros2_control.xacro (robot description, xacro)
@@ -90,4 +90,44 @@
         <state_interface name="velocity"/>
       </joint>
+      <joint name="right_finger_joint">
+        <command_interface name="position"/>
+        <state_interface name="position"/>
+        <state_interface name="velocity"/>
+      </joint>
+      <joint name="right_external_rod_joint">
+        <param name="mimic">right_finger_joint</param>
+        <param name="multiplier">-1</param>
+        <command_interface name="position"/>
+        <state_interface name="position"/>
+        <state_interface name="velocity"/>
+      </joint>
+      <joint name="right_fingertip_joint">
+        <param name="mimic">right_finger_joint</param>
+        <param name="multiplier">-1</param>
+        <command_interface name="position"/>
+        <state_interface name="position"/>
+        <state_interface name="velocity"/>
+      </joint>
+      <joint name="left_finger_joint">
+        <param name="mimic">right_finger_joint</param>
+        <param name="multiplier">-1</param>
+        <command_interface name="position"/>
+        <state_interface name="position"/>
+        <state_interface name="velocity"/>
+      </joint>
+      <joint name="left_external_rod_joint">
+        <param name="mimic">right_finger_joint</param>
+        <param name="multiplier">-1</param>
+        <command_interface name="position"/>
+        <state_interface name="position"/>
+        <state_interface name="velocity"/>
+      </joint>
+      <joint name="left_fingertip_joint">
+        <param name="mimic">right_finger_joint</param>
+        <param name="multiplier">-1</param>
+        <command_interface name="position"/>
+        <state_interface name="position"/>
+        <state_interface name="velocity"/>
+      </joint>
       <joint name="left_wheel_joint">
         <command_interface name="velocity">

File: explorer_on_wheelchair/description/urdf/simulation.urdf.xacro (robot description, xacro)
@@ -6,4 +6,6 @@
   <xacro:include filename="$(find ros2_control_explorer)/description/urdf/explorer_old_description.urdf.xacro" />
   <xacro:explorer_old_description/>
+  <xacro:include filename="$(find gripper_pincette)/description/urdf/gripper_pincette_description.urdf.xacro"/>
+  <xacro:gripper_pincette/>
   <link name="fixation">
     <visual>
@@ -35,4 +37,21 @@
     <child link="base_link"/>
   </joint>
+    <joint name="joint_6" type="revolute">
+    <parent link="link_5"/>
+    <child link="structure"/>
+    <origin xyz="0 0.090 0.083" rpy="${-(65*pi)/180} 0 0"/>
+    <axis xyz="0 0 1"/>
+    <limit effort="1000.0" lower="${-pi}" upper="${pi}" velocity="2.5"/>
+  </joint>
+  <joint name="joint-ft_frame" type="fixed">
+    <parent link="structure"/>
+    <child link="ft_frame"/>
+    <origin xyz="0.011 0 0.15" rpy="0 0 0"/>
+  </joint>
+  <joint name="joint-tool" type="fixed">
+    <parent link="ft_frame"/>
+    <child link="tool0"/>
+    <origin xyz="0 0 0" rpy="0 0 0"/>
+  </joint>
   <xacro:include filename="$(find explorer_on_wheelchair)/description/ros2_control/simulation.ros2_control.xacro" />
   <xacro:simulation_ros2_control name="simulation"/>

Commit message: (fix): change inertia

File: explorer_on_wheelchair/description/ros2_control/simulation.ros2_control.xacro (robot description, xacro)
@@ -137,4 +137,5 @@
         <state_interface name="position"/>
         <state_interface name="velocity"/>
+        <state_interface name="effort"/>
       </joint>
       <joint name="right_wheel_joint">
@@ -145,4 +146,5 @@
         <state_interface name="position"/>
         <state_interface name="velocity"/>
+        <state_interface name="effort"/>
       </joint>
     </ros2_control>

File: explorer_on_wheelchair/description/urdf/simulation.urdf.xacro (robot description, xacro)
@@ -22,7 +22,7 @@
     </collision>
     <inertial>
-      <origin rpy="0 0 0" xyz="0 0 0"/>
-      <mass value="1"/>
-      <inertia ixx="1" ixy="0" ixz="0" iyy="1" iyz="0" izz="1"/>
+      <origin rpy="0 0 0" xyz="0 -0.03 -0.03"/>
+      <mass value="0.5"/>
+      <inertia ixx="0.00084166666" ixy="0" ixz="0" iyy="0.000675" iyz="0" izz="0.00084166666"/>
     </inertial>
   </link>
