Commit message: (fix): change disabled_simulator to explorer_on_wheelchair

File: explorer_on_wheelchair/description/gazebo/simulation.gazebo.xacro (robot description, xacro)
@@ -5,5 +5,5 @@
     <gazebo>
       <plugin filename="libgazebo_ros2_control.so" name="gazebo_ros2_control_simulation">
-        <parameters>$(find disabled_simulator)/config/simulation_controllers.yaml</parameters>
+        <parameters>$(find explorer_on_wheelchair)/config/simulation_controllers.yaml</parameters>
       </plugin>
     </gazebo>

File: explorer_on_wheelchair/description/urdf/simulation.urdf.xacro (robot description, xacro)
@@ -10,5 +10,5 @@
       <origin rpy="0 0 0" xyz="0 0 0"/>
       <geometry>
-        <mesh filename="file://$(find disabled_simulator)/description/meshes/visual/fixation.dae" scale="0.001 0.001 0.001"/>
+        <mesh filename="file://$(find explorer_on_wheelchair)/description/meshes/visual/fixation.dae" scale="0.001 0.001 0.001"/>
       </geometry>
     </visual>
@@ -16,5 +16,5 @@
       <origin rpy="0 0 0" xyz="0 0 0"/>
       <geometry>
-        <mesh filename="file://$(find disabled_simulator)/description/meshes/collision/fixation.stl" scale="0.001 0.001 0.001"/>
+        <mesh filename="file://$(find explorer_on_wheelchair)/description/meshes/collision/fixation.stl" scale="0.001 0.001 0.001"/>
       </geometry>
     </collision>
@@ -35,7 +35,7 @@
     <child link="base_link"/>
   </joint>
-  <xacro:include filename="$(find disabled_simulator)/description/ros2_control/simulation.ros2_control.xacro" />
+  <xacro:include filename="$(find explorer_on_wheelchair)/description/ros2_control/simulation.ros2_control.xacro" />
   <xacro:simulation_ros2_control name="simulation"/>
-  <xacro:include filename="$(find disabled_simulator)/description/gazebo/simulation.gazebo.xacro" />
+  <xacro:include filename="$(find explorer_on_wheelchair)/description/gazebo/simulation.gazebo.xacro" />
   <xacro:simulation_gazebo/>
 </robot>

Commit message: (fix): use ignition only

File: explorer_on_wheelchair/description/gazebo/simulation.gazebo.xacro (robot description, xacro)
@@ -4,8 +4,141 @@
     <!-- ros_control plugin -->
     <gazebo>
-      <plugin filename="libgazebo_ros2_control.so" name="gazebo_ros2_control_simulation">
+      <plugin filename="ign_ros2_control-system" name="ign_ros2_control::IgnitionROS2ControlPlugin">
         <parameters>$(find explorer_on_wheelchair)/config/simulation_controllers.yaml</parameters>
       </plugin>
     </gazebo>
+    <gazebo reference="base_link">
+      <visual>
+          <material>
+              <diffuse>1 1 1 1</diffuse>
+          </material>
+      </visual>
+    </gazebo>
+    <gazebo reference="link_1">
+      <visual>
+          <material>
+              <diffuse>1 1 1 1</diffuse>
+          </material>
+      </visual>
+    </gazebo>
+    <gazebo reference="link_2">
+      <visual>
+          <material>
+              <diffuse>1 1 1 1</diffuse>
+          </material>
+      </visual>
+    </gazebo>
+    <gazebo reference="link_3">
+      <visual>
+          <material>
+              <diffuse>1 1 1 1</diffuse>
+          </material>
+      </visual>
+    </gazebo>
+    <gazebo reference="link_4">
+      <visual>
+          <material>
+              <diffuse>1 1 1 1</diffuse>
+          </material>
+      </visual>
+    </gazebo>
+    <gazebo reference="link_5">
+      <visual>
+          <material>
+              <diffuse>1 1 1 1</diffuse>
+          </material>
+      </visual>
+    </gazebo>
+    <gazebo reference="structure">
+      <visual>
+          <material>
+              <diffuse>1 1 1 1</diffuse>
+          </material>
+      </visual>
+    </gazebo>
+    <gazebo reference="motor">
+      <visual>
+          <material>
+              <diffuse>1 1 1 1</diffuse>
+          </material>
+      </visual>
+    </gazebo>
+    <gazebo reference="palm_top_shell">
+      <visual>
+          <material>
+              <diffuse>1 1 1 1</diffuse>
+          </material>
+      </visual>
+    </gazebo>
+    <gazebo reference="right_finger_first_phalanx">
+      <visual>
+          <material>
+              <diffuse>1 1 1 1</diffuse>
+          </material>
+      </visual>
+    </gazebo>
+    <gazebo reference="right_external_rod">
+      <visual>
+          <material>
+              <diffuse>1 1 1 1</diffuse>
+          </material>
+      </visual>
+    </gazebo>
+    <gazebo reference="right_finger_last_phalanx">
+      <visual>
+          <material>
+              <diffuse>1 1 1 1</diffuse>
+          </material>
+      </visual>
+    </gazebo>
+    <gazebo reference="left_finger_first_phalanx">
+      <visual>
+          <material>
+              <diffuse>1 1 1 1</diffuse>
+          </material>
+      </visual>
+    </gazebo>
+    <gazebo reference="left_external_rod">
+      <visual>
+          <material>
+              <diffuse>1 1 1 1</diffuse>
+          </material>
+      </visual>
+    </gazebo>
+    <gazebo reference="left_finger_last_phalanx">
+      <visual>
+          <material>
+              <diffuse>1 1 1 1</diffuse>
+          </material>
+      </visual>
+    </gazebo>
+      <gazebo reference="foam_seat">
+      <visual>
+          <material>
+              <diffuse>1 1 1 1</diffuse>
+          </material>
+      </visual>
+    </gazebo>
+    <gazebo reference="foam_backrest">
+      <visual>
+          <material>
+              <diffuse>1 1 1 1</diffuse>
+          </material>
+      </visual>
+    </gazebo>
+    <gazebo reference="foam_headrest">
+      <visual>
+          <material>
+              <diffuse>1 1 1 1</diffuse>
+          </material>
+      </visual>
+    </gazebo>
+    <gazebo reference="fixation">
+      <visual>
+          <material>
+              <diffuse>1 1 1 1</diffuse>
+          </material>
+      </visual>
+    </gazebo>
   </xacro:macro>
 </robot>

File: explorer_on_wheelchair/description/ros2_control/simulation.ros2_control.xacro (robot description, xacro)
@@ -4,5 +4,5 @@
     <ros2_control name="${name}" type="system">
       <hardware>
-          <plugin>gazebo_ros2_control/GazeboSystem</plugin>
+          <plugin>ign_ros2_control/IgnitionSystem</plugin>
       </hardware>
       <joint name="joint_1">
@@ -90,8 +90,9 @@
         <state_interface name="velocity"/>
       </joint>
-      <joint name="right_finger_joint">
+<joint name="right_finger_joint">
         <command_interface name="position"/>
         <state_interface name="position"/>
         <state_interface name="velocity"/>
+        <state_interface name="effort"/>
       </joint>
       <joint name="right_external_rod_joint">
@@ -101,4 +102,5 @@
         <state_interface name="position"/>
         <state_interface name="velocity"/>
+        <state_interface name="effort"/>
       </joint>
       <joint name="right_fingertip_joint">
@@ -108,4 +110,5 @@
         <state_interface name="position"/>
         <state_interface name="velocity"/>
+        <state_interface name="effort"/>
       </joint>
       <joint name="left_finger_joint">
@@ -115,4 +118,5 @@
         <state_interface name="position"/>
         <state_interface name="velocity"/>
+        <state_interface name="effort"/>
       </joint>
       <joint name="left_external_rod_joint">
@@ -122,4 +126,5 @@
         <state_interface name="position"/>
         <state_interface name="velocity"/>
+        <state_interface name="effort"/>
       </joint>
       <joint name="left_fingertip_joint">
@@ -129,4 +134,5 @@
         <state_interface name="position"/>
         <state_interface name="velocity"/>
+        <state_interface name="effort"/>
       </joint>
       <joint name="left_wheel_joint">

Commit message: (fix): add camera and world

File: explorer_on_wheelchair/description/gazebo/simulation.gazebo.xacro (robot description, xacro)
@@ -141,4 +141,25 @@
       </visual>
     </gazebo>
+    <gazebo reference="camera_explorer">
+      <sensor name="camera" type="camera">
+        <camera>
+          <optical_frame_id>camera_explorer</optical_frame_id>
+          <horizontal_fov>1.047</horizontal_fov>
+          <image>
+              <width>640</width>
+              <height>400</height>
+          </image>
+          <clip>
+              <near>0.05</near>
+              <far>100</far>
+          </clip>
+        </camera>
+        <always_on>1</always_on>
+        <update_rate>30</update_rate>
+        <visualize>true</visualize>
+        <topic>camera</topic>
+        <enable_metrics>false</enable_metrics>
+      </sensor>
+    </gazebo>
   </xacro:macro>
 </robot>

File: explorer_on_wheelchair/description/urdf/simulation.urdf.xacro (robot description, xacro)
@@ -8,4 +8,5 @@
   <xacro:include filename="$(find gripper_pincette)/description/urdf/gripper_pincette_description.urdf.xacro"/>
   <xacro:gripper_pincette/>
+  <link name="camera_explorer"/>
   <link name="fixation">
     <visual>
@@ -37,8 +38,8 @@
     <child link="base_link"/>
   </joint>
-    <joint name="joint_6" type="revolute">
+  <joint name="joint_6" type="revolute">
     <parent link="link_5"/>
     <child link="structure"/>
-    <origin xyz="0 0.090 0.083" rpy="${-(65*pi)/180} 0 0"/>
+    <origin xyz="0 0.090 0.083" rpy="0 ${(65*pi)/180} ${pi/2}"/>
     <axis xyz="0 0 1"/>
     <limit effort="1000.0" lower="${-pi}" upper="${pi}" velocity="2.5"/>
@@ -48,4 +49,9 @@
     <child link="ft_frame"/>
     <origin xyz="0.011 0 0.15" rpy="0 0 0"/>
+  </joint>
+  <joint name="camera_joint" type="fixed">
+    <parent link="structure"/>
+    <child link="camera_explorer"/>
+    <origin xyz="0.011 0 0.105" rpy="0 ${-pi/2} 0"/>
   </joint>
   <joint name="joint-tool" type="fixed">

Commit message: (feat): add head and wheelchair control with xbox controller

File: explorer_on_wheelchair/description/gazebo/simulation.gazebo.xacro (robot description, xacro)
@@ -162,4 +162,25 @@
       </sensor>
     </gazebo>
+    <gazebo reference="user_vision_camera">
+      <sensor name="camera" type="camera">
+        <camera>
+          <optical_frame_id>user_vision_camera</optical_frame_id>
+          <horizontal_fov>1.047</horizontal_fov>
+          <image>
+              <width>1200</width>
+              <height>600</height>
+          </image>
+          <clip>
+              <near>0.05</near>
+              <far>100</far>
+          </clip>
+        </camera>
+        <always_on>1</always_on>
+        <update_rate>30</update_rate>
+        <visualize>true</visualize>
+        <topic>user_vision</topic>
+        <enable_metrics>false</enable_metrics>
+      </sensor>
+    </gazebo>
   </xacro:macro>
 </robot>

File: explorer_on_wheelchair/description/ros2_control/simulation.ros2_control.xacro (robot description, xacro)
@@ -154,4 +154,20 @@
         <state_interface name="effort"/>
       </joint>
+      <joint name="left_right_head_joint">
+        <command_interface name="position">
+          <param name="min">{-60*pi/180}</param>
+          <param name="max">{60*pi/180}</param>
+        </command_interface>
+        <state_interface name="position"/>
+        <state_interface name="velocity"/>
+      </joint>
+      <joint name="up_down_head_joint">
+        <command_interface name="position">
+          <param name="min">{-70*pi/180}</param>
+          <param name="max">{40*pi/180}</param>
+        </command_interface>
+        <state_interface name="position"/>
+        <state_interface name="velocity"/>
+      </joint>
     </ros2_control>
   </xacro:macro>

File: explorer_on_wheelchair/description/urdf/simulation.urdf.xacro (robot description, xacro)
@@ -9,4 +9,5 @@
   <xacro:gripper_pincette/>
   <link name="camera_explorer"/>
+  <link name="user_vision_camera"/>
   <link name="fixation">
     <visual>
@@ -55,4 +56,9 @@
     <origin xyz="0.011 0 0.105" rpy="0 ${-pi/2} 0"/>
   </joint>
+  <joint name="eye_camera_joint" type="fixed">
+    <parent link="head_up_down"/>
+    <child link="user_vision_camera"/>
+    <origin xyz="0.1 0 0" rpy="0 0 0"/>
+  </joint>
   <joint name="joint-tool" type="fixed">
     <parent link="ft_frame"/>
