Commit message: feat : update simulation to work with POC2 version

File: explorer_on_wheelchair/description/urdf/simulation.urdf.xacro (robot description, xacro)
@@ -4,6 +4,13 @@
   <xacro:include filename="$(find ros2_control_wheelchair)/description/urdf/wheelchair_description.urdf.xacro" />
   <xacro:wheelchair/>
-  <xacro:include filename="$(find ros2_control_explorer)/description/urdf/explorer_POC1_description.urdf.xacro" />
-  <xacro:explorer_old_description/>
+  <xacro:include filename="$(find ros2_control_explorer)/description/urdf/explorer_POC2_description.urdf.xacro"/>
+  <joint name="joint_6" type="revolute">
+    <parent link="link_5"/>
+    <child link="structure"/>
+    <origin xyz="0 0.1555 -0.027" rpy="${pi/2} ${pi} ${pi}"/>
+    <axis xyz="0 0 1"/>
+    <limit effort="1000.0" lower="-2.97" upper="2.97" velocity="10"/>
+  </joint>
+  <xacro:explorer_POC2_description/>
   <xacro:include filename="$(find gripper_pincette)/description/urdf/gripper_pincette_description.urdf.xacro"/>
   <xacro:gripper_pincette/>
@@ -39,11 +46,4 @@
     <child link="base_link"/>
   </joint>
-  <joint name="joint_6" type="revolute">
-    <parent link="link_5"/>
-    <child link="structure"/>
-    <origin xyz="0 0.090 0.083" rpy="0 ${(65*pi)/180} ${pi/2}"/>
-    <axis xyz="0 0 1"/>
-    <limit effort="1000.0" lower="${-pi}" upper="${pi}" velocity="2.5"/>
-  </joint>
   <joint name="joint-ft_frame" type="fixed">
     <parent link="structure"/>
